Commit message: Removes the propery pi, as it is included globally within xacro in kinetic

File: ur_description/urdf/ur10.urdf.xacro (robot description, xacro)
@@ -7,5 +7,4 @@
   <xacro:include filename="$(find ur_description)/urdf/ur.transmission.xacro" />
   <xacro:include filename="$(find ur_description)/urdf/ur.gazebo.xacro" />
-  <xacro:property name="pi" value="3.14159265" />
   <!-- Inertia parameters -->
   <xacro:property name="base_mass" value="4.0" />  <!-- This mass might be incorrect -->

File: ur_description/urdf/ur3.urdf.xacro (robot description, xacro)
@@ -6,5 +6,4 @@
   <xacro:include filename="$(find ur_description)/urdf/ur.transmission.xacro" />
   <xacro:include filename="$(find ur_description)/urdf/ur.gazebo.xacro" />
-  <xacro:property name="pi" value="3.14159265" />
   <!-- Inertia parameters -->
   <xacro:property name="base_mass" value="2.0" />  <!-- This mass might be incorrect -->

File: ur_description/urdf/ur5.urdf.xacro (robot description, xacro)
@@ -3,5 +3,4 @@
   <xacro:include filename="$(find ur_description)/urdf/ur.transmission.xacro" />
   <xacro:include filename="$(find ur_description)/urdf/ur.gazebo.xacro" />
-  <xacro:property name="pi" value="3.14159265" />
   <!-- Inertia parameters -->
   <xacro:property name="base_mass" value="4.0" />  <!-- This mass might be incorrect -->

Commit message: Adds the possibility to have precise and non-precise collision geometry

File: ur_description/urdf/ur10.urdf.xacro (robot description, xacro)
@@ -58,5 +58,6 @@
 		 wrist_1_lower_limit:=${-pi}    wrist_1_upper_limit:=${pi}
 		 wrist_2_lower_limit:=${-pi}    wrist_2_upper_limit:=${pi}
-		 wrist_3_lower_limit:=${-pi}    wrist_3_upper_limit:=${pi}">
+		 wrist_3_lower_limit:=${-pi}    wrist_3_upper_limit:=${pi}
+     precise_collision:=true">
     <link name="${prefix}base_link" >
       <visual>
@@ -68,9 +69,19 @@
         </material>
       </visual>
-      <collision>
-        <geometry>
-          <mesh filename="package://ur_description/meshes/ur10/collision/base.stl"/>
-        </geometry>
-      </collision>
+      <xacro:if value="${precise_collision}">
+        <collision>
+          <geometry>
+            <mesh filename="package://ur_description/meshes/ur10/collision/base.stl"/>
+          </geometry>
+        </collision>
+      </xacro:if>
+      <xacro:unless value="${precise_collision}">
+        <collision>
+          <origin xyz="0.0 -0.005 0.02" rpy="0 0 0" />
+          <geometry>
+            <box size="0.16 0.17 0.04"/>
+          </geometry>
+        </collision>
+      </xacro:unless>
       <xacro:cylinder_inertial radius="0.075" length="0.038" mass="${base_mass}">
         <origin xyz="0.0 0.0 0.0" rpy="0 0 0" />
@@ -99,9 +110,19 @@
         </material>
       </visual>
-      <collision>
-        <geometry>
-          <mesh filename="package://ur_description/meshes/ur10/collision/shoulder.stl"/>
-        </geometry>
-      </collision>
+      <xacro:if value="${precise_collision}">
+        <collision>
+          <geometry>
+            <mesh filename="package://ur_description/meshes/ur10/collision/shoulder.stl"/>
+          </geometry>
+        </collision>
+      </xacro:if>
+      <xacro:unless value="${precise_collision}">
+        <collision>
+          <origin xyz="0.0 0.015 0.0" rpy="0 0 0" />
+          <geometry>
+            <cylinder radius="0.10" length="0.18"/>
+          </geometry>
+        </collision>
+      </xacro:unless>
       <xacro:cylinder_inertial radius="0.075" length="0.178" mass="${shoulder_mass}">
         <origin xyz="0.0 0.0 0.0" rpy="0 0 0" />
@@ -130,9 +151,19 @@
         </material>
       </visual>
-      <collision>
-        <geometry>
-          <mesh filename="package://ur_description/meshes/ur10/collision/upperarm.stl"/>
-        </geometry>
-      </collision>
+      <xacro:if value="${precise_collision}">
+        <collision>
+          <geometry>
+            <mesh filename="package://ur_description/meshes/ur10/collision/upperarm.stl"/>
+          </geometry>
+        </collision>
+      </xacro:if>
+      <xacro:unless value="${precise_collision}">
+        <collision>
+          <origin xyz="0.0 -0.045 0.3" rpy="0 0 0" />
+          <geometry>
+            <cylinder radius="0.09" length="0.75"/>
+          </geometry>
+        </collision>
+      </xacro:unless>
       <xacro:cylinder_inertial radius="0.075" length="${-ur10_a2}" mass="${upper_arm_mass}">
         <origin xyz="0.0 0.0 ${-ur10_a2/2.0}" rpy="0 0 0" />
@@ -161,9 +192,19 @@
         </material>
       </visual>
-      <collision>
-        <geometry>
-          <mesh filename="package://ur_description/meshes/ur10/collision/forearm.stl"/>
-        </geometry>
-      </collision>
+      <xacro:if value="${precise_collision}">
+        <collision>
+          <geometry>
+            <mesh filename="package://ur_description/meshes/ur10/collision/forearm.stl"/>
+          </geometry>
+        </collision>
+      </xacro:if>
+      <xacro:unless value="${precise_collision}">
+        <collision>
+          <origin xyz="0.0 0.0 0.28" rpy="0 0 0" />
+          <geometry>
+            <cylinder radius="0.07" length="0.68"/>
+          </geometry>
+        </collision>
+      </xacro:unless>
       <xacro:cylinder_inertial radius="0.075" length="${-ur10_a3}" mass="${forearm_mass}">
         <origin xyz="0.0 0.0 ${-ur10_a3/2.0}" rpy="0 0 0" />
@@ -192,9 +233,19 @@
         </material>
       </visual>
-      <collision>
-        <geometry>
-          <mesh filename="package://ur_description/meshes/ur10/collision/wrist1.stl"/>
-        </geometry>
-      </collision>
+      <xacro:if value="${precise_collision}">
+        <collision>
+          <geometry>
+            <mesh filename="package://ur_description/meshes/ur10/collision/wrist1.stl"/>
+          </geometry>
+        </collision>
+      </xacro:if>
+      <xacro:unless value="${precise_collision}">
+        <collision>
+          <origin xyz="0.0 0.11 0.005" rpy="0 0 0" />
+          <geometry>
+            <cylinder radius="0.05" length="0.12"/>
+          </geometry>
+        </collision>
+      </xacro:unless>
       <xacro:cylinder_inertial radius="0.075" length="0.12" mass="${wrist_1_mass}">
         <origin xyz="0.0 0.0 0.0" rpy="0 0 0" />
@@ -223,9 +274,19 @@
         </material>
       </visual>
-      <collision>
-        <geometry>
-          <mesh filename="package://ur_description/meshes/ur10/collision/wrist2.stl"/>
-        </geometry>
-      </collision>
+      <xacro:if value="${precise_collision}">
+        <collision>
+          <geometry>
+            <mesh filename="package://ur_description/meshes/ur10/collision/wrist2.stl"/>
+          </geometry>
+        </collision>
+      </xacro:if>
+      <xacro:unless value="${precise_collision}">
+        <collision>
+          <origin xyz="0.0 0.005 0.115" rpy="1.5708 0 0" />
+          <geometry>
+            <cylinder radius="0.05" length="0.13"/>
+          </geometry>
+        </collision>
+      </xacro:unless>
       <xacro:cylinder_inertial radius="0.075" length="0.12" mass="${wrist_2_mass}">
         <origin xyz="0.0 0.0 0.0" rpy="0 0 0" />
@@ -254,9 +315,19 @@
         </material>
       </visual>
-      <collision>
-        <geometry>
-          <mesh filename="package://ur_description/meshes/ur10/collision/wrist3.stl"/>
-        </geometry>
-      </collision>
+      <xacro:if value="${precise_collision}">
+        <collision>
+          <geometry>
+            <mesh filename="package://ur_description/meshes/ur10/collision/wrist3.stl"/>
+          </geometry>
+        </collision>
+      </xacro:if>
+      <xacro:unless value="${precise_collision}">
+        <collision>
+          <origin xyz="0.0 0.078 0.0" rpy="1.5708 0 0" />
+          <geometry>
+            <cylinder radius="0.05" length="0.033"/>
+          </geometry>
+        </collision>
+      </xacro:unless>
       <xacro:cylinder_inertial radius="0.075" length="0.12" mass="${wrist_3_mass}">
         <origin xyz="0.0 0.0 0.0" rpy="0 0 0" />

Commit message: Improves the rough collision to be a bit more accurate

File: ur_description/urdf/ur10.urdf.xacro (robot description, xacro)
@@ -203,5 +203,17 @@
           <origin xyz="0.0 0.0 0.28" rpy="0 0 0" />
           <geometry>
-            <cylinder radius="0.07" length="0.68"/>
+            <cylinder radius="0.045" length="0.58"/>
+          </geometry>
+        </collision>
+        <collision>
+          <origin xyz="0.0 0.0 0.575" rpy="1.5708 0 0 " />
+          <geometry>
+            <cylinder radius="0.045" length="0.12"/>
+          </geometry>
+        </collision>
+        <collision>
+          <origin xyz="0.0 0.0 0.0" rpy="1.5708 0 0 " />
+          <geometry>
+            <cylinder radius="0.06" length="0.13"/>
           </geometry>
         </collision>

Commit message: Removes useless collision geometry

File: ur_description/urdf/ur10.urdf.xacro (robot description, xacro)
@@ -351,14 +351,6 @@
       <origin xyz="0.0 ${wrist_3_length} 0.0" rpy="0.0 0.0 ${pi/2.0}" />
     </joint>
-    <link name="${prefix}ee_link">
-      <collision>
-        <geometry>
-          <box size="0.01 0.01 0.01"/>
-        </geometry>
-        <origin rpy="0 0 0" xyz="-0.01 0 0"/>
-      </collision>
-    </link>
+    <link name="${prefix}ee_link" />
     <xacro:ur_arm_transmission prefix="${prefix}" />
-    <xacro:ur_arm_gazebo prefix="${prefix}" />
     <!-- ROS base_link to UR 'Base' Coordinates transform -->
     <link name="${prefix}base"/>
